Commit message: Corrected the link visualization error

File: continuum_rb/urdf/rb_model.urdf (robot description, URDF)
Before this commit: robot continuum_robot, 9 links, 8 joints
Links:
- added link link0; visual cylinder length=0.1 radius=0.3
Joints:
- added joint joint0: type floating, parent base_link, child link0
